Commit message: Turtlebot urdf model was changed

File: ros/src/turtlebot3/turtlebot3_description/urdf/turtlebot3_burger.gazebo.xacro (robot description, xacro)
@@ -123,10 +123,11 @@
    <!-- camera -->
   <gazebo reference="camera_link">
+    <material>Gazebo/DarkGrey</material>
     <sensor type="camera" name="camera1">
       <always_on>true</always_on>
       <visualize>$(arg camera_visual)</visualize>
-      <update_rate>30.0</update_rate>
+      <update_rate>5.0</update_rate>
       <camera>
-        <horizontal_fov>1.3962634</horizontal_fov>
+        <horizontal_fov>1.39626</horizontal_fov>
         <image>
           <width>640</width>

File: ros/src/turtlebot3/turtlebot3_description/urdf/turtlebot3_burger.urdf.xacro (robot description, xacro)
@@ -4,7 +4,7 @@
   <xacro:include filename="$(find turtlebot3_description)/urdf/turtlebot3_burger.gazebo.xacro"/>
     <!-- Mount and camera parameters -->
-  <xacro:property name="r200_cam_offset_px" value="-0.017" />
-  <xacro:property name="r200_cam_offset_py" value="0.024" />
-  <xacro:property name="r200_cam_offset_pz" value="0.005" />
+  <xacro:property name="r200_cam_offset_px" value="0.032" />
+  <xacro:property name="r200_cam_offset_py" value="0.000" />
+  <xacro:property name="r200_cam_offset_pz" value="0.171" />
   <link name="base_footprint"/>
   <joint name="base_joint" type="fixed">
@@ -120,5 +120,5 @@
     <parent link="base_link"/>
     <child link="base_scan"/>
-    <origin xyz="-0.032 0 0.171" rpy="0 0 0"/>
+    <origin xyz="-0.032 0 0.171" rpy="${-M_PI*0.5} 0 0"/>
   </joint>
   <link name="base_scan">
@@ -161,9 +161,10 @@
       <origin xyz="0 0 0" rpy="${M_PI/2} 0 ${M_PI/2}"/>
         <geometry>
-         <mesh filename="package://turtlebot3_description/meshes/sensors/r200.dae" />
+         <mesh filename="package://turtlebot3_description/meshes/sensors/astra.dae" scale="0.001 0.001 0.001"/>
         </geometry>
+        <material name="dark"/>
     </visual>
     <inertial>
-      <mass value="0.564" />
+      <mass value="0.01" />
         <origin xyz="0 0 0" />
         <inertia ixx="0.003881243" ixy="0.0" ixz="0.0"
